Commit message: comment out capsule geom for yourdf support

File: models/rby1a/urdf/model.urdf (robot description, URDF)
Before this commit: robot RB_Y1_V1.0.1, 34 links, 33 joints
Links:
- link link_left_arm_0: geometry visual mesh filename=./meshes/LINK_14.dae
- link link_left_arm_1: geometry visual mesh filename=./meshes/LINK_15.dae
- link link_left_arm_2: geometry visual mesh filename=./meshes/LINK_16.dae
- link link_left_arm_3: geometry visual mesh filename=./meshes/LINK_17.dae
- link link_left_arm_4: geometry visual mesh filename=./meshes/LINK_18.dae
- link link_left_arm_5: geometry visual mesh filename=./meshes/LINK_19.dae
- link link_right_arm_0: geometry visual mesh filename=./meshes/LINK_7.dae
- link link_right_arm_1: geometry visual mesh filename=./meshes/LINK_8.dae
- link link_right_arm_2: geometry visual mesh filename=./meshes/LINK_9.dae
- link link_right_arm_3: geometry visual mesh filename=./meshes/LINK_10.dae
- link link_right_arm_4: geometry visual mesh filename=./meshes/LINK_11.dae
- link link_right_arm_5: geometry visual mesh filename=./meshes/LINK_12.dae
- link link_torso_0: geometry visual mesh filename=./meshes/LINK_1.dae
- link link_torso_1: geometry visual mesh filename=./meshes/LINK_2.dae
- link link_torso_2: geometry visual mesh filename=./meshes/LINK_3.dae
- link link_torso_4: geometry visual mesh filename=./meshes/LINK_5.dae
- link link_torso_5: geometry visual mesh filename=./meshes/LINK_6.dae
